Commit message: Local g3 tooling edits carried onto gen4 (EXPERIMENTS.md, eval/plot scripts, hoop URDF)
Uncommitted working-tree edits from the g3 work, committed as-is so the gen4
branch is self-contained: EXPERIMENTS.md log, summarize_evals / plot_epoch_rewards
/ plot_gen2_by_subject and their tests, retarget_contact, smplx_pose,
generate_hoop_urdf + hoop_bball.urdf, test_eval_cfgs.

Co-Authored-By: Claude Fable 5.1 <noreply@anthropic.com>

File: isaacgym/src/intermimic/data/assets/objects/hoop_bball.urdf (robot description, URDF)
Before this commit: robot hoop_bball, 1 links, 0 joints
Links:
- link hoop: geometry collision box size=0.04 1.10 0.80; collision box size=0.14 0.14 3.7340
